File: Si_FET_Adapter.brd (EAGLE design)
At the start: 21.6 x 15.2 mm, 13 parts

Commit message: 発注
Parts:
- moved C1 33.7 mm to (4.45, 12.7)
- moved C2 33.7 mm to (16.5, 12.7)
- moved FB1 33.7 mm to (13.3, 3.17)
- moved FB2 33.7 mm to (3.17, 3.17)
- moved Q1 33.7 mm to (15.2, 7.62)
- moved Q2 33.7 mm to (6.35, 7.62)
- moved R1 33.7 mm to (12.4, 12.7)
- moved R2 33.7 mm to (8.57, 12.7)
- moved TP1 33.7 mm to (17.8, 1.27)
- moved TP2 33.7 mm to (10.2, 1.27)
- moved TP3 33.7 mm to (5.08, 1.27)
- moved TP4 33.7 mm to (2.54, 1.27)
- moved TP5 33.7 mm to (12.7, 1.27)
Other:
- board size 21.6 x 15.2 mm -> 21 x 15.2 mm
